File: UGOKU-One.kicad_pcb (KiCad board)
At the start: 2 copper layers, 63 x 63 mm, 56 parts, among them CN1 Conn_01x04, CN2 Conn_01x04, CN3 Conn_01x04, CN4 CAN, J2 Conn_02x03_Odd_Even, J3 Conn_01x02_Male, J4 PA10, J6 Conn_01x04, SW1 PF1, SW2 RESET, SW3 SW_Push_DPDT, SW5 SW_Push_DPDT, T1 PTS_1.5_2, T2 PTS_1.5_2, T3 PTS_1.5_2, U1 M78AR5-1, U2 NUCLEO-F303K8, U4 TB67H303HG, U5 TB67H303HG, U6 MCP2562-E_SN, U7 ESP32-WROOM-32

Commit message: commit iroiro
Parts:
- removed C11, C13, C2, C3, C9: 0.1μF, Capacitor_SMD:C_0805_2012Metric
- removed C12, C5: 47μF, Capacitor_THT:CP_Radial_D6.3mm_P2.50mm
- removed CN4: CAN, Connector_JST:JST_XA_B03B-XASK-1_1x03_P2.50mm_Vertical
- removed J6: Conn_01x04, Connector_PinSocket_2.54mm:PinSocket_1x04_P2.54mm_Vertical
- removed JP4: Jumper_NC_Dual, Jumper:SolderJumper-3_P2.0mm_Open_TrianglePad1.0x1.5mm
- removed MH1, MH2, MH3, MH4: MountingHole_3.2mm_M3, MountingHole:MountingHole_3.2mm_M3
- removed MJP1, MJP2: Jumper, Jumper:SolderJumper-2_P1.3mm_Open_TrianglePad1.0x1.5mm
- removed R13, R7: 51kΩ, Resistor_SMD:R_0603_1608Metric
- removed R2, R3: 10kΩ, Resistor_SMD:R_0603_1608Metric
- removed R9: 10k, Resistor_SMD:R_0603_1608Metric
- removed T1, T2: PTS_1.5_2, MultiBoardMini_Libraries:PTS_1.5_2
- removed U2: NUCLEO-F303K8, MultiBoardMini_Libraries:MODULE_NUCLEO-F303K8
- removed U4, U5: TB67H303HG, MultiBoardMini_Libraries:TO100P2930X465X1937-25
- removed U6: MCP2562-E_SN, MultiBoardMini_Libraries:SOIC127P600X175-8N
- added BZ1: Buzzer, Buzzer_Beeper:Buzzer_12x9.5RM7.6, F.Cu at (42.0, -10.0)
- added P1: USB_C_Plug_USB2.0, Connector_USB:USB_C_Receptacle_GCT_USB4105-xx-A_16P_TopMnt_Horizontal, F.Cu at (25.4, 13.3)
- added Q1: 2SC2712, Package_TO_SOT_SMD:SOT-23, F.Cu at (55.0, -4.67)
- added T5: MultiBoardMini_Libraries:PTS_1.5_2, UGOKU-One_Libraries:PTS_1.5_2, F.Cu at (24.3, 43.1)
- added U3: TB67H450FNG_EL, Package_SO:HSOP-8-1EP_3.9x4.9mm_P1.27mm_EP2.3x2.3mm, F.Cu at (14.5, 40.3)
- added U8: TB67H450FNG_EL, Package_SO:HSOP-8-1EP_3.9x4.9mm_P1.27mm_EP2.3x2.3mm, F.Cu at (14.5, 46.9)
- C1: value 0.1μF -> 10μF
- C10: value 3.3μF -> 22μF
- CN1, CN2, CN3: footprint Connector_JST:JST_XA_B04B-XASK-1_1x04_P2.50mm_Vertical -> UGOKU-One_Libraries:har-flexicon_2.54_4pin
- R1: value 120Ω -> 10k; moved to F.Cu
- R4: value 3.3k -> 510
- R5, R6: value 3.3k -> 1k
- U1: value M78AR5-1 -> K7803-500R3; moved to F.Cu
- U7: moved to F.Cu
- moved R1 45.6 mm to (59.5, -5.82), turned to 0 degrees
- moved C1 26.1 mm to (1.73, 11.0), turned to 0 degrees
- moved SW3 18.1 mm to (16.0, 5.00)
- moved SW4 18.1 mm to (15.5, -1.00)
- moved U1 4.75 mm to (0.54, 9.50), turned to 180 degrees
- turned U7 to 0 degrees
Connections:
- C1 pad 1: +5V -> PWR
- C10 pad 1: +5V -> +3V3
- CN1 pad 3: Net-(CN1-Pin_3) -> unconnected-(CN1-Pin_3-Pad3)
- CN1 pad 4: Net-(CN1-Pin_4) -> unconnected-(CN1-Pin_4-Pad4)
- CN2 pad 3: Net-(CN2-Pin_3) -> unconnected-(CN2-Pin_3-Pad3)
- CN2 pad 4: Net-(CN2-Pin_4) -> unconnected-(CN2-Pin_4-Pad4)
- CN3 pad 3: Net-(CN3-Pin_3) -> unconnected-(CN3-Pin_3-Pad3)
- CN3 pad 4: Net-(CN3-Pin_4) -> unconnected-(CN3-Pin_4-Pad4)
- J2 pad 3: Net-(J2-Pin_3) -> PWR
- J2 pad 4: Net-(J2-Pin_3) -> PWR
- J2 pad 5: Net-(J2-Pin_5) -> unconnected-(J2-Pin_5-Pad5)
- J2 pad 6: Net-(J2-Pin_6) -> unconnected-(J2-Pin_6-Pad6)
- L2 pad 2: Net-(CN2-Pin_4) -> unconnected-(L2-A-Pad2)
- L3 pad 2: Net-(CN2-Pin_3) -> unconnected-(L3-A-Pad2)
- R1 pad 2: Net-(CN4-Pin_3) -> unconnected-(R1-Pad2)
- SW1 pad 2: Net-(U2A-PF1) -> unconnected-(SW1-Pad2)
- SW2 pad 2: Net-(U2A-NRST_1) -> unconnected-(SW2-Pad2)
- U1 pad 1: Net-(J4-Pin_1) -> PWR
- U1 pad 3: +5V -> +3V3
- U7 pad 27: Net-(U2A-PA9) -> unconnected-(U7-IO16-Pad27)
- U7 pad 28: Net-(U2A-PA10) -> unconnected-(U7-IO17-Pad28)
- U7 pad 34: Net-(J6-Pin_2) -> unconnected-(U7-RXD0/IO3-Pad34)
- U7 pad 35: Net-(J6-Pin_1) -> unconnected-(U7-TXD0/IO1-Pad35)
Routing:
- net GND: track 233.5 -> 0.00 mm, vias 36 -> 0
- net +5V: track 158.5 -> 0.00 mm, vias 2 -> 0
- net +3V3: track 138.7 -> 0.00 mm, vias 3 -> 0
- net PWR: track 135.4 -> 0.00 mm
- net Net-(SW5-B-Pad2): track 57.4 -> 0.00 mm
- net Net-(U2A-PB5): track 56.0 -> 0.00 mm, vias 4 -> 0
- net Net-(U5-OUT2A): track 49.8 -> 0.00 mm
- net Net-(U4-OUT1A): track 49.6 -> 0.00 mm
- net Net-(CN2-Pin_3): track 46.8 -> 0.00 mm
- net Net-(U2A-NRST_1): track 43.7 -> 0.00 mm
- net Net-(U5-OUT1A): track 43.2 -> 0.00 mm
- net Net-(U4-OUT2A): track 42.9 -> 0.00 mm
- net Net-(U2A-PB4): track 42.1 -> 0.00 mm, vias 3 -> 0
- net Net-(U2A-PB1): track 41.9 -> 0.00 mm, vias 1 -> 0
- net Net-(CN2-Pin_4): track 40.8 -> 0.00 mm, vias 2 -> 0
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
Commit message: make concept
Parts:
- removed CN1, CN2, CN3: Conn_01x04, UGOKU-One_Libraries:har-flexicon_2.54_4pin
- added BT1: Battery, 0_UGOKU-One_Lib:BAT_2481, B.Cu at (0.15, 0.05)
- added J4: 14110413001000, 0_UGOKU-One_Lib:14110413001000, F.Cu at (-11.0, 5.13)
- added J5: 14110413001000, 0_UGOKU-One_Lib:14110413001000, F.Cu at (-11.1, -15.2)
- added J6: 14110413001000, 0_UGOKU-One_Lib:14110413001000, F.Cu at (-11.1, -5.03)
- added T4: PTS_1.5_2, 0_UGOKU-One_Lib:PTS_1.5_2, F.Cu at (11.0, 25.8)
- T5: footprint UGOKU-One_Libraries:PTS_1.5_2 -> 0_UGOKU-One_Lib:PTS_1.5_2
- moved R1 49.1 mm to (10.7, -0.27)
- moved U8 49.0 mm to (-22.5, 14.8)
- moved BZ1 44.8 mm to (0.79, 7.69)
- moved T5 39.5 mm to (-11.4, 26.0)
- moved Q1 33.3 mm to (21.7, -2.85)
- moved U3 26.7 mm to (22.7, 14.9)
- moved P1 7.28 mm to (25.7, 6.05)

Commit message: add PD
Parts:
- removed J3: Conn_01x02_Male, Connector_JST:JST_XA_B02B-XASK-1_1x02_P2.50mm_Vertical
- removed R12: 10k, Resistor_SMD:R_0603_1608Metric
- removed SW3: SW_Push_DPDT, MultiBoardMini_Libraries:SSSS213202
- removed SW4: ~, Button_Switch_SMD:SW_Push_1P1T_NO_Vertical_Wuerth_434133025816
- removed T3: PTS_1.5_2, MultiBoardMini_Libraries:PTS_1.5_2
- added C11: 22μF, Capacitor_SMD:C_0805_2012Metric, F.Cu at (45.5, 15.7)
- added C12: 100nF, Capacitor_SMD:C_0402_1005Metric, F.Cu at (79.5, 3.59)
- added C13: 4.7uF, Capacitor_SMD:C_0805_2012Metric, F.Cu at (72.9, -2.00)
- added C14: 1uF, Capacitor_SMD:C_0805_2012Metric, F.Cu at (72.9, 1.01)
- added C15: 1uF, Capacitor_SMD:C_0805_2012Metric, F.Cu at (72.9, 4.02)
- added C16: 1uF, Capacitor_SMD:C_0805_2012Metric, F.Cu at (72.9, 7.03)
- added C17: 1uF, Capacitor_SMD:C_0201_0603Metric, F.Cu at (79.3, -0.02)
- added C18: 1uF, Capacitor_SMD:C_0201_0603Metric, F.Cu at (79.3, 1.73)
- added C4: 10μF, Capacitor_SMD:C_0805_2012Metric, F.Cu at (45.5, -2.36)
- added C5: 10μF, Capacitor_SMD:C_0805_2012Metric, F.Cu at (45.5, 0.65)
- added C6: 10μF, Capacitor_SMD:C_0805_2012Metric, F.Cu at (45.5, 3.66)
- added C7: 10μF, Capacitor_SMD:C_0805_2012Metric, F.Cu at (45.5, 6.67)
- added C8: 10μF, Capacitor_SMD:C_0805_2012Metric, F.Cu at (45.5, 9.68)
- added C9: 10μF, Capacitor_SMD:C_0805_2012Metric, F.Cu at (45.5, 12.7)
- added D9: ESDA25P35-1U1M, 0_UGOKU-One_Lib:TVS_ESDA25P35-1U1M, F.Cu at (80.2, -2.20)
- added J1: USB_C_Receptacle_USB2.0_16P, Connector_USB:USB_C_Receptacle_GCT_USB4105-xx-A_16P_TopMnt_Horizontal, F.Cu at (53.6, 1.42)
- added JP4: Jumper_NC_Dual, Jumper:SolderJumper-3_P2.0mm_Open_TrianglePad1.0x1.5mm, F.Cu at (56.2, 15.2)
- added JP5: Jumper_NC_Dual, Jumper:SolderJumper-3_P2.0mm_Open_TrianglePad1.0x1.5mm, F.Cu at (56.2, 19.0)
- added Q2: SS8050, Package_TO_SOT_SMD:SOT-23, F.Cu at (50.2, 8.53)
- added Q3: SS8050, Package_TO_SOT_SMD:SOT-23, F.Cu at (50.2, 13.2)
- added Q4: SI2319CDS, Package_TO_SOT_SMD:SOT-23, F.Cu at (50.2, 17.8)
- added R13: 10k, Resistor_SMD:R_0603_1608Metric, F.Cu at (41.3, -2.61)
- added R14: 10k, Resistor_SMD:R_0603_1608Metric, F.Cu at (41.3, -0.10)
- added R15: 10k, Resistor_SMD:R_0603_1608Metric, F.Cu at (41.3, 2.41)
- added R16: 10k, Resistor_SMD:R_0603_1608Metric, F.Cu at (41.3, 4.92)
- added R17: 5.1k, Resistor_SMD:R_0603_1608Metric, F.Cu at (41.3, 7.43)
- added R18: 10k, Resistor_SMD:R_0603_1608Metric, F.Cu at (41.3, 9.94)
- added R19: 10k, Resistor_SMD:R_0603_1608Metric, F.Cu at (41.3, 12.4)
- added R20: 10k, Resistor_SMD:R_0603_1608Metric, F.Cu at (41.3, 15.0)
- added R21: 100k, Resistor_SMD:R_0402_1005Metric, F.Cu at (41.3, 17.5)
- added R22: 22k, Resistor_SMD:R_0402_1005Metric, F.Cu at (76.6, -2.51)
- added R23: 100, Resistor_SMD:R_0402_1005Metric, F.Cu at (76.6, -0.52)
- added R24: 1k, Resistor_SMD:R_0402_1005Metric, F.Cu at (76.6, 1.47)
- added R25: 4.7k, Resistor_SMD:R_0402_1005Metric, F.Cu at (76.6, 3.46)
- added R26: 4.7K, Resistor_SMD:R_0402_1005Metric, F.Cu at (76.6, 5.45)
- added U2: CP2102N-A02-GQFN28, 0_UGOKU-One_Lib:QFN50P500X500X80-29N, F.Cu at (56.8, 9.76)
- added U5: STUSB4500QTR, Package_DFN_QFN:QFN-24-1EP_4x4mm_P0.5mm_EP2.7x2.7mm, F.Cu at (62.6, -0.71)
- added U6: XC6206P272MR, Package_TO_SOT_SMD:SOT-23-3, F.Cu at (62.3, 15.8)
- D1: value D -> ESDA25P35-1U1M; footprint Diode_SMD:D_SOD-123 -> 0_UGOKU-One_Lib:TVS_ESDA25P35-1U1M
- moved D1 64.0 mm to (61.9, 19.5), turned to 0 degrees
Connections:
- C1 pad 1: PWR -> 5V
- J2 pad 3: PWR -> SERVO_PWR
- J2 pad 4: PWR -> SERVO_PWR
- P1 pad A5: unconnected-(P1-CC-PadA5) -> Net-(P1-CC)
- P1 pad A6: unconnected-(P1-D+-PadA6) -> Net-(D4-A2)
- P1 pad A7: unconnected-(P1-D--PadA7) -> Net-(D3-A2)
- P1 pad S1: unconnected-(P1-SHIELD-PadS1) -> GND
- U1 pad 1: PWR -> 5V
- U3 pad 5: PWR -> MOT_PWR
- U7 pad 3: Net-(D1-A) -> EN
- U7 pad 34: unconnected-(U7-RXD0/IO3-Pad34) -> RXD
- U7 pad 35: unconnected-(U7-TXD0/IO1-Pad35) -> TXD
- U8 pad 5: PWR -> MOT_PWR

Commit message: V1 Rough Layout
Parts:
- removed BZ1: Buzzer, Buzzer_Beeper:Buzzer_12x9.5RM7.6
- removed C12: 100nF, Capacitor_SMD:C_0402_1005Metric
- removed C13: 4.7uF, Capacitor_SMD:C_0805_2012Metric
- removed C14, C15, C16: 1uF, Capacitor_SMD:C_0805_2012Metric
- removed C17, C18: 1uF, Capacitor_SMD:C_0201_0603Metric
- removed the C4 at (45.5, -2.36)
- removed D1, D9: ESDA25P35-1U1M, 0_UGOKU-One_Lib:TVS_ESDA25P35-1U1M
- removed J1: USB_C_Receptacle_USB2.0_16P, Connector_USB:USB_C_Receptacle_GCT_USB4105-xx-A_16P_TopMnt_Horizontal
- removed the J4 at (2.54, 18.0)
- removed JP4, JP5: Jumper_NC_Dual, Jumper:SolderJumper-3_P2.0mm_Open_TrianglePad1.0x1.5mm
- removed Q1: 2SC2712, Package_TO_SOT_SMD:SOT-23
- removed Q4: SI2319CDS, Package_TO_SOT_SMD:SOT-23
- removed R1, R20: 10k, Resistor_SMD:R_0603_1608Metric
- removed R21: 100k, Resistor_SMD:R_0402_1005Metric
- removed R22: 22k, Resistor_SMD:R_0402_1005Metric
- removed R23: 100, Resistor_SMD:R_0402_1005Metric
- removed R24: 1k, Resistor_SMD:R_0402_1005Metric
- removed R25: 4.7k, Resistor_SMD:R_0402_1005Metric
- removed R26: 4.7K, Resistor_SMD:R_0402_1005Metric
- removed SW2: RESET, MultiBoardMini_Libraries:SW_TL3301FF160QG
- removed U6: XC6206P272MR, Package_TO_SOT_SMD:SOT-23-3
- removed U7: ESP32-WROOM-32, RF_Module:ESP32-WROOM-32
- added D2: LESD5D5.0CT1G, Diode_SMD:D_SOD-523, F.Cu at (20.4, 4.00)
- added D3: LESD5D5.0CT1G, Diode_SMD:D_SOD-523, F.Cu at (20.4, 6.45)
- added D4: LESD5D5.0CT1G, Diode_SMD:D_SOD-523, F.Cu at (20.4, 8.90)
- added D5: SS54, Diode_SMD:D_SMA, F.Cu at (9.00, 5.50)
- added D6: SS54, Diode_SMD:D_SMA, F.Cu at (-21.0, 8.00)
- added D7: SS54, Diode_SMD:D_SMA, F.Cu at (9.00, 9.50)
- added H1: MountingHole, MountingHole:MountingHole_3.2mm_M3, F.Cu at (-30.0, -30.0)
- added H2: MountingHole, MountingHole:MountingHole_3.2mm_M3, F.Cu at (30.0, -20.0)
- added H3: MountingHole, MountingHole:MountingHole_3.2mm_M3, F.Cu at (-30.0, 30.0)
- added H4: MountingHole, MountingHole:MountingHole_3.2mm_M3, F.Cu at (30.0, 30.0)
- added J3: Conn_02x03_Odd_Even, Connector_PinHeader_2.54mm:PinHeader_2x03_P2.54mm_Vertical_SMD, F.Cu at (-1.04, 5.53)
- added SW4: SW_Push, Button_Switch_SMD:SW_Push_1P1T_NO_Vertical_Wuerth_434133025816, F.Cu at (0.93, -11.9)
- added SW6: SW_Push, Button_Switch_SMD:SW_Push_1P1T_NO_Vertical_Wuerth_434133025816, F.Cu at (0.93, -6.42)
- added T6: PTS_1.5_2, 0_UGOKU-One_Lib:PTS_1.5_2, F.Cu at (-9.50, 27.5)
- added U4: K7805M-1000R3, 0_UGOKU-One_Lib:M78AR, F.Cu at (8.54, 17.5)
- C1, C5: value 10μF -> 22μF; footprint Capacitor_SMD:C_0805_2012Metric -> Capacitor_SMD:C_0603_1608Metric
- C10, C11: footprint Capacitor_SMD:C_0805_2012Metric -> Capacitor_SMD:C_0603_1608Metric
- C4: moved to F.Cu
- C6: value 10μF -> 0.1μF; footprint Capacitor_SMD:C_0805_2012Metric -> Capacitor_SMD:C_0603_1608Metric
- C7, C8: value 10μF -> 0.1uF; footprint Capacitor_SMD:C_0805_2012Metric -> Capacitor_SMD:C_0603_1608Metric
- J2: value Conn_02x03_Odd_Even -> SERVO; footprint Connector_PinHeader_2.54mm:PinHeader_2x03_P2.54mm_Vertical -> Connector_PinHeader_2.54mm:PinHeader_2x03_P2.54mm_Vertical_SMD
- SW1: footprint MultiBoardMini_Libraries:SW_TL3301FF160QG -> Button_Switch_SMD:SW_Push_1P1T_NO_Vertical_Wuerth_434133025816
- U1: value K7803-500R3 -> AMS1117-3.3; footprint MultiBoardMini_Libraries:M78AR -> Package_TO_SOT_SMD:SOT-223-3_TabPin2
- U5: value STUSB4500QTR -> ESP32-WROOM-32E; footprint Package_DFN_QFN:QFN-24-1EP_4x4mm_P0.5mm_EP2.7x2.7mm -> RF_Module:ESP32-WROOM-32D
- moved U5 51.0 mm to (15.0, -19.0)
- moved C4 46.1 mm to (27.6, 25.0)
- moved U2 37.4 mm to (21.1, -1.50)
- moved SW1 34.3 mm to (0.93, -18.4)
- moved L1 29.2 mm to (30.5, -11.0)
- moved L2 29.2 mm to (33.8, -11.0)
- moved L3 29.2 mm to (37.0, -11.0)
- moved R4 29.2 mm to (30.5, -7.25)
- moved R5 29.2 mm to (33.8, -7.25)
- moved R6 29.2 mm to (37.0, -7.25)
- moved P1 26.7 mm to (17.0, 31.3), turned to 0 degrees
- moved Q2 26.1 mm to (27.1, -3.50)
- moved U3 26.1 mm to (-3.42, 14.9)
- moved Q3 25.0 mm to (28.1, 1.50)
- moved J2 24.0 mm to (-12.0, 13.5)
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Connections:
- net Net-(D2-A2) renamed USB_5V
- C7 pad 1: Net-(U7-IO0) -> GND
- C7 pad 2: GND -> IO0
- C9 pad 1: Net-(D10-K) -> PWR
- J2 pad 5: unconnected-(J2-Pin_5-Pad5) -> SERVO2
- J2 pad 6: unconnected-(J2-Pin_6-Pad6) -> SERVO1
- L2 pad 2: unconnected-(L2-A-Pad2) -> LED1
- L3 pad 2: unconnected-(L3-A-Pad2) -> LED2
- U3 pad 2: unconnected-(U3-IN2-Pad2) -> MD1_IN2
- U3 pad 3: unconnected-(U3-IN1-Pad3) -> MD1_IN1
- U5 pad 1: Net-(J1-CC1) -> GND
- U5 pad 10: GND -> unconnected-(U5-IO25-Pad10)
- U5 pad 13: unconnected-(U5-ADDR1-Pad13) -> SERVO1
- U5 pad 14: unconnected-(U5-POWER_OK3-Pad14) -> MD2_IN1
- U5 pad 15: unconnected-(U5-GPIO-Pad15) -> GND
- U5 pad 16: Net-(U5-VBUS_EN_SNK) -> MD2_IN2
- U5 pad 18: Net-(U5-VBUS_VS_DISCH) -> unconnected-(U5-NC-Pad18)
- U5 pad 2: Net-(J1-CC1) -> +3V3
- U5 pad 21: Net-(U5-VREG_1V2) -> unconnected-(U5-NC-Pad21)
- U5 pad 23: +2V7 -> SERVO2
- U5 pad 24: Net-(D1-K) -> LED1
- U5 pad 25: GND -> IO0
- U5 pad 3: unconnected-(U5-NC-Pad3) -> EN
- U5 pad 4: Net-(J1-CC2) -> unconnected-(U5-SENSOR_VP-Pad4)
- U5 pad 5: Net-(J1-CC2) -> unconnected-(U5-SENSOR_VN-Pad5)
- U5 pad 7: Net-(U5-SCL) -> unconnected-(U5-IO35-Pad7)
- U5 pad 8: Net-(U5-SDA) -> unconnected-(U5-IO32-Pad8)
- U8 pad 2: unconnected-(U8-IN2-Pad2) -> MD2_IN2
- U8 pad 3: unconnected-(U8-IN1-Pad3) -> MD2_IN1
Other:
- board size 63 x 63 mm -> 70 x 70 mm
- board text added: "UGOKU One Ver1.0.0 UGOKU Lab 2025-4"
- board text removed: "+5V"
- board text removed: "0.1μF"
- board text removed: "10kΩ"
- board text removed: "120Ω"
- board text removed: "47μF"
- board text removed: "51kΩ"
- board text removed: "5V"
- board text removed: "5V PWR"
- board text removed: "6-32V"
- board text removed: "CAN"
- board text removed: "ESP BOOT"
- board text removed: "ESP EN"
- board text removed: "ESP32 WRITE"
- board text removed: "ESP32-WROOM-32E"
- board text removed: "GND"
- board text removed: "H"
- board text removed: "L"
- board text removed: "M1 ON"
- board text removed: "M2 ON"
- board text removed: "MCP2562"
- board text removed: "Nucleo-F303K8"
- board text removed: "PA0"
- board text removed: "PA1"
- board text removed: "PA3"
- board text removed: "PA4"
- board text removed: "PB3"
- board text removed: "PB6"
- board text removed: "PB7"
- board text removed: "PF1"
- board text removed: "RESET"
- board text removed: "RX"
- board text removed: "SERVO POWER SOURCE"
- board text removed: "TX"
- board text removed: "UGOKU One Ver0.4.5 UGOKU Lab 2024-4"
