File: UGOKU-One.kicad_sch (KiCad schematic)
At the start: 52 parts, among them J2 Conn_02x03_Odd_Even, J2 PA10, J3 Conn_01x02_Male, J6 Conn_01x04, SW1 PF1, SW2 RESET, SW3 SW_Push_DPDT, SW5 SW_Push_DPDT, T1 PTS_1.5_2, T3 PTS_1.5_2, U2 NUCLEO-F303K8, U3 M78AR5-1, U4 TB67H303HG, U5 TB67H303HG, U6 MCP2562-E_SN, U7 ESP32-WROOM-32

Commit message: commit iroiro
Parts:
- removed C10, C2, C4 (x4): 0.1μF, Capacitor_SMD:C_0805_2012Metric, symbol Device:C
- removed C5 (x2): 47μF, Capacitor_THT:CP_Radial_D6.3mm_P2.50mm, symbol Device:CP
- removed CAN1: CAN, Connector_JST:JST_XA_B03B-XASK-1_1x03_P2.50mm_Vertical, symbol Connector_Generic:Conn_01x03
- removed J2: PA10, Connector_PinHeader_2.54mm:PinHeader_1x03_P2.54mm_Vertical, symbol Connector_Generic:Conn_01x03
- removed J6: Conn_01x04, Connector_PinSocket_2.54mm:PinSocket_1x04_P2.54mm_Vertical, symbol Connector_Generic:Conn_01x04
- removed JP1: Jumper_NC_Dual, Jumper:SolderJumper-3_P2.0mm_Open_TrianglePad1.0x1.5mm, symbol Device:Jumper_NC_Dual
- removed MJP1 (x2): Jumper, Jumper:SolderJumper-2_P1.3mm_Open_TrianglePad1.0x1.5mm, symbol Device:Jumper
- removed R2 (x2): 10kΩ, Resistor_SMD:R_0603_1608Metric, symbol Device:R
- removed R3 (x2): 51kΩ, Resistor_SMD:R_0603_1608Metric, symbol Device:R
- removed R9: 10k, Resistor_SMD:R_0603_1608Metric, symbol Device:R
- removed T1 (x2): PTS_1.5_2, MultiBoardMini_Libraries:PTS_1.5_2, symbol pts_1.5_2:PTS_1.5_2
- removed U2: NUCLEO-F303K8, MultiBoardMini_Libraries:MODULE_NUCLEO-F303K8, symbol NUCLEO-F303K8:NUCLEO-F303K8
- removed U4, U5: TB67H303HG, MultiBoardMini_Libraries:TO100P2930X465X1937-25, symbol TB67H303HG:TB67H303HG
- removed U6: MCP2562-E_SN, MultiBoardMini_Libraries:SOIC127P600X175-8N, symbol MCP2562-E_SN:MCP2562-E_SN
- added BZ1: Buzzer, Buzzer_Beeper:Buzzer_12x9.5RM7.6, symbol Device:Buzzer
- added P1: USB_C_Plug_USB2.0, Connector_USB:USB_C_Receptacle_GCT_USB4105-xx-A_16P_TopMnt_Horizontal, symbol Connector:USB_C_Plug_USB2.0
- added Q1: 2SC2712, Package_TO_SOT_SMD:SOT-23, symbol Transistor_BJT:2SC4213
- added T4: PTS_1.5_2, MultiBoardMini_Libraries:PTS_1.5_2, symbol pts_1.5_2:PTS_1.5_2
- added T5: MultiBoardMini_Libraries:PTS_1.5_2, UGOKU-One_Libraries:PTS_1.5_2, symbol pts_1.5_2:PTS_1.5_2
- added U3, U8: TB67H450FNG_EL, Package_SO:HSOP-8-1EP_3.9x4.9mm_P1.27mm_EP2.3x2.3mm, symbol TB67H450FNG:TB67H450FNG_EL
- C1: value 0.1μF -> 10μF
- C9: value 3.3μF -> 22μF
- ENC/IO_1, ENC/IO_2, IO_1: footprint Connector_JST:JST_XA_B04B-XASK-1_1x04_P2.50mm_Vertical -> UGOKU-One_Libraries:har-flexicon_2.54_4pin
- R1: value 120Ω -> 10k
- U3: value M78AR5-1 -> K7803-500R3
Connections:
- net +3V3: now also C9.1, U3.3 (Vout); no longer C1.1
- net +5V: now also BZ1.1 (-), U3.4 (VREF), U8.4 (VREF); no longer C9.1, U3.3 (Vout)
- net GND: now also Q1.2 (E), U3.1 (GND), U3.7 (RS), U3.9 (GND), U8.1 (GND), U8.7 (RS), U8.9 (GND)
- net PWR: now also C1.1, J2.3 (Pin_3), J2.4 (Pin_4), U3.1 (Vin), U3.5 (VM), U8.5 (VM)
- net at PA1.2 (A): no longer ENC/IO_2.4 (Pin_4)
- net at ENC/IO_2.3 (Pin_3): no longer PA2.2 (A)
- net at R1.1: now also Q1.1 (B)
- new net: T4.P$1, U3.6 (OUT1)
- new net: T4.P$2, U3.8 (OUT2)
- new net: T5.P$1, U8.6 (OUT1)
- new net: T5.P$2, U8.8 (OUT2)
- new net: BZ1.2 (+), Q1.3 (C)
- new net: P1.A1 (GND), P1.A12 (GND), P1.B1 (GND), P1.B12 (GND)
- new net: P1.A4 (VBUS), P1.A9 (VBUS), P1.B4 (VBUS), P1.B9 (VBUS)
- no-connect marks 39 -> 31
Other:
- note removed: "V0.4.4"
- moved on the sheet: C9, D1, ENC/IO_1, ENC/IO_2, IO_1, J2, J3, JP1, JP2, JP3, PA1, PA2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

Commit message: modify usb, power
Parts:
- removed D1: D, Diode_SMD:D_SOD-123, symbol Device:D
- removed ENC/IO_1, ENC/IO_2, IO_1: Conn_01x04, UGOKU-One_Libraries:har-flexicon_2.54_4pin, symbol Connector_Generic:Conn_01x04
- removed J3: Conn_01x02_Male, Connector_JST:JST_XA_B02B-XASK-1_1x02_P2.50mm_Vertical, symbol Connector:Conn_01x02_Male
- removed R10: 10k, Resistor_SMD:R_0603_1608Metric, symbol Device:R
- removed SW3: SW_Push_DPDT, MultiBoardMini_Libraries:SSSS213202, symbol Switch:SW_Push_DPDT
- removed T3: PTS_1.5_2, MultiBoardMini_Libraries:PTS_1.5_2, symbol pts_1.5_2:PTS_1.5_2
- added BT1: Battery, 0_UGOKU-One_Lib:BAT_2481, symbol Device:Battery
- added C11: 22μF, Capacitor_SMD:C_0805_2012Metric, symbol Device:C
- added C2, C3: C, symbol Device:C
- added C4, C5, C6, C7, C8, C9: 10μF, Capacitor_SMD:C_0805_2012Metric, symbol Device:C
- added D2, D3, D4: D_TVS, symbol Device:D_TVS
- added D5, D6, D7, D8: D, symbol Device:D
- added H1: MountingHole, symbol Mechanical:MountingHole
- added J4, J5, J6: 14110413001000, 0_UGOKU-One_Lib:14110413001000, symbol 0_14110413001000:14110413001000
- added JP4, JP5: Jumper_NC_Dual, Jumper:SolderJumper-3_P2.0mm_Open_TrianglePad1.0x1.5mm, symbol Device:Jumper_NC_Dual
- added Q2, Q3: SS8050, Package_TO_SOT_SMD:SOT-23, symbol Transistor_BJT:SS8050
- added R13, R14, R15, R16, R18, R19, R20: 10k, Resistor_SMD:R_0603_1608Metric, symbol Device:R
- added R17: 5.1k, Resistor_SMD:R_0603_1608Metric, symbol Device:R
- added SW6: SW_Push, symbol Switch:SW_Push
- added U2: CP2102N-A02-GQFN28, 0_UGOKU-One_Lib:QFN50P500X500X80-29N, symbol 0_CP2102N:CP2102N-A02-GQFN28
- added U4: K7805-1000R3, MultiBoardMini_Libraries:M78AR, symbol Liner-regulator_AOKI:NJM_TO-252
- SW4: value ~ -> SW_Push; footprint Button_Switch_SMD:SW_Push_1P1T_NO_Vertical_Wuerth_434133025816 -> (none)
- T4: footprint MultiBoardMini_Libraries:PTS_1.5_2 -> 0_UGOKU-One_Lib:PTS_1.5_2
- T5: footprint UGOKU-One_Libraries:PTS_1.5_2 -> 0_UGOKU-One_Lib:PTS_1.5_2
- renumbered C9 to C10, PWR1 to L1, PA1 to L2, PA2 to L3, U3 to U1
Connections:
- net +3V3: now also C2.1, C3.1, C5.1, C6.1, R13.2, R20.2, U2.6 (VDD), U2.7 (VREGIN)
- net GND: now also P1.A1 (GND), P1.A12 (GND), P1.B1 (GND), P1.B12 (GND), P1.S1 (SHIELD), SW4.2, BT1.2 (-), C11.2, C2.2, C3.2, C4.2, C5.2, C6.2, C7.2, C8.1, C9.2, D2.1 (A1), D3.1 (A1), D4.1 (A1), J4.2, J5.2, J6.2, R15.1, R16.1, R17.1, SW6.1, U2.29 (GND), U2.3 (GND), U4.2 (GND); no longer SW4.1
- net PWR: now also JP4.3, JP5.3; no longer C1.1, J2.3 (Pin_3), J2.4 (Pin_4), U1.1 (Vin), U3.5 (VM), U8.5 (VM)
- net at JP3.2: now also J6.1
- net at JP2.2: now also J5.1
- net at JP1.2: now also J4.1
- net at U7.25 (IO0): now also SW4.1, C7.1
- net EN: now reaches U7.3 (EN)
- net EN: now also C4.1, C8.2, Q2.3 (C), R20.1, SW6.2; no longer SW4.2
- net RXD: now reaches U7.34 (RXD0/IO3)
- net RXD: now also U2.25 (RXD)
- net TXD: now reaches U7.35 (TXD0/IO1)
- net TXD: now also U2.26 (TXD)
- net at P1.A4 (VBUS), P1.A9 (VBUS), P1.B4 (VBUS)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: now also D2.2 (A2), D5.2 (A), R14.2
- net at P1.A5 (CC): now also R17.2
- net at P1.A6 (D+): now also D4.2 (A2), U2.4 (D+)
- net at P1.A7 (D-): now also D3.2 (A2), U2.5 (D-)
- new net: C11.1, D8.2 (A), U4.3 (Vout)
- new net: R14.1, R15.2, U2.8 (VBUS)
- new net: R16.2, U2.11 (~{SUSPEND})
- new net: Q2.1 (B), R18.1
- new net: Q2.2 (E), R19.2, U2.24 (RTS)
- new net: Q3.2 (E), R18.2, U2.28 (DTR)
- new net: R13.1, U2.9 (~{RST})
- new net: Q3.1 (B), R19.1
- new net 5V: C1.1, D6.1 (K), D7.1 (K), D8.1 (K), JP4.1, JP5.1, U1.1 (Vin)
- new net BAT_5V: BT1.1 (+), D6.2 (A)
- new net EXT_PWR: C9.1, U4.1 (Vin)
- new net IO0: Q3.3 (C)
- new net MOT_PWR: JP4.2, U3.5 (VM), U8.5 (VM)
- new net SERVO_PWR: J2.3 (Pin_3), J2.4 (Pin_4), JP5.2
- new net USB_5V: D5.1 (K), D7.2 (A)
- no-connect marks 31 -> 45
Other:
- moved on the sheet: C1, C10, L1, L2, L3, P1, R4, R5, R6, U1

Commit message: add PD
Parts:
- added C12: 100nF, Capacitor_SMD:C_0402_1005Metric, symbol Device:C
- added C13: 4.7uF, Capacitor_SMD:C_0805_2012Metric, symbol Device:C
- added C14, C15, C16: 1uF, Capacitor_SMD:C_0805_2012Metric, symbol Device:C
- added C17, C18: 1uF, Capacitor_SMD:C_0201_0603Metric, symbol Device:C
- added D1, D9: ESDA25P35-1U1M, 0_UGOKU-One_Lib:TVS_ESDA25P35-1U1M, symbol Diode:BZM55Bxx
- added D10, D11: D, symbol Device:D
- added J1: USB_C_Receptacle_USB2.0_16P, Connector_USB:USB_C_Receptacle_GCT_USB4105-xx-A_16P_TopMnt_Horizontal, symbol Connector:USB_C_Receptacle_USB2.0_16P
- added Q4: SI2319CDS, Package_TO_SOT_SMD:SOT-23, symbol Simulation_SPICE:PMOS
- added R21: 100k, Resistor_SMD:R_0402_1005Metric, symbol Device:R
- added R22: 22k, Resistor_SMD:R_0402_1005Metric, symbol Device:R
- added R23: 100, Resistor_SMD:R_0402_1005Metric, symbol Device:R
- added R24: 1k, Resistor_SMD:R_0402_1005Metric, symbol Device:R
- added R25: 4.7k, Resistor_SMD:R_0402_1005Metric, symbol Device:R
- added R26: 4.7K, Resistor_SMD:R_0402_1005Metric, symbol Device:R
- added U5: STUSB4500QTR, Package_DFN_QFN:QFN-24-1EP_4x4mm_P0.5mm_EP2.7x2.7mm, symbol Interface_USB:STUSB4500QTR
- added U6: XC6206P272MR, Package_TO_SOT_SMD:SOT-23-3, symbol Liner-regulator_AOKI:NJM_TO-252
Connections:
- net +3V3: now also C18.2, U6.1 (Vin)
- net EXT_PWR: now also D11.2 (A); no longer C9.1, U4.1 (Vin)
- net GND: now also C13.2, C14.1, C15.1, C16.1, C17.1, C18.1, D1.2 (A), D9.2 (A), J1.A1 (GND), J1.A12 (GND), J1.B1 (GND), J1.B12 (GND), J1.S1 (SHIELD), U5.10 (GND), U5.25 (GND), U6.2 (GND); no longer P1.A1 (GND), P1.A12 (GND), P1.B1 (GND), P1.B12 (GND)
- net PWR: now also C9.1, U4.1 (Vin), D10.1 (K), D11.1 (K)
- new net: R25.1, U5.7 (SCL)
- new net: C12.2, R23.1
- new net: Q4.2 (G), R21.1, R22.2, R23.2
- new net: J1.A5 (CC1), U5.1 (CC1DB), U5.2 (CC1)
- new net: R22.1, U5.16 (VBUS_EN_SNK)
- new net: R24.1, U5.18 (VBUS_VS_DISCH)
- new net: C16.2, U5.21 (VREG_1V2)
- new net: C13.1, C14.2, D1.1 (K), J1.A4 (VBUS), J1.A9 (VBUS), J1.B4 (VBUS), J1.B9 (VBUS), Q4.3 (S), R21.2, R24.2, U5.24 (VDD)
- new net: J1.B5 (CC2), U5.4 (CC2), U5.5 (CC2DB)
- new net: R26.1, U5.8 (SDA)
- new net: P1.A1 (GND), P1.A12 (GND), P1.B1 (GND), P1.B12 (GND)
- new net +2V7: C15.2, C17.2, R25.2, R26.2, U5.23 (VREG_2V7), U6.3 (Vout)
- new net PD_PWR: C12.1, D10.2 (A), D9.1 (K), Q4.1 (D)
- no-connect marks 45 -> 51
Other:
- moved on the sheet: J4, J5, J6, JP1, JP2, JP3, SW1, SW2

Commit message: V1 Rough Layout
Parts:
- removed BZ1: Buzzer, Buzzer_Beeper:Buzzer_12x9.5RM7.6, symbol Device:Buzzer
- removed C12: 100nF, Capacitor_SMD:C_0402_1005Metric, symbol Device:C
- removed C13: 4.7uF, Capacitor_SMD:C_0805_2012Metric, symbol Device:C
- removed C14, C15, C16: 1uF, Capacitor_SMD:C_0805_2012Metric, symbol Device:C
- removed C17, C18: 1uF, Capacitor_SMD:C_0201_0603Metric, symbol Device:C
- removed C4: 10μF, Capacitor_SMD:C_0805_2012Metric, symbol Device:C
- removed D1, D9: ESDA25P35-1U1M, 0_UGOKU-One_Lib:TVS_ESDA25P35-1U1M, symbol Diode:BZM55Bxx
- removed D10, D11, D5, D6, D7, D8: D, symbol Device:D
- removed J1: USB_C_Receptacle_USB2.0_16P, Connector_USB:USB_C_Receptacle_GCT_USB4105-xx-A_16P_TopMnt_Horizontal, symbol Connector:USB_C_Receptacle_USB2.0_16P
- removed JP4, JP5: Jumper_NC_Dual, Jumper:SolderJumper-3_P2.0mm_Open_TrianglePad1.0x1.5mm, symbol Device:Jumper_NC_Dual
- removed Q1: 2SC2712, Package_TO_SOT_SMD:SOT-23, symbol Transistor_BJT:2SC4213
- removed Q4: SI2319CDS, Package_TO_SOT_SMD:SOT-23, symbol Simulation_SPICE:PMOS
- removed R1, R20: 10k, Resistor_SMD:R_0603_1608Metric, symbol Device:R
- removed R21: 100k, Resistor_SMD:R_0402_1005Metric, symbol Device:R
- removed R22: 22k, Resistor_SMD:R_0402_1005Metric, symbol Device:R
- removed R23: 100, Resistor_SMD:R_0402_1005Metric, symbol Device:R
- removed R24: 1k, Resistor_SMD:R_0402_1005Metric, symbol Device:R
- removed R25: 4.7k, Resistor_SMD:R_0402_1005Metric, symbol Device:R
- removed R26: 4.7K, Resistor_SMD:R_0402_1005Metric, symbol Device:R
- removed SW2: RESET, MultiBoardMini_Libraries:SW_TL3301FF160QG, symbol Switch:SW_Push
- removed U5: STUSB4500QTR, Package_DFN_QFN:QFN-24-1EP_4x4mm_P0.5mm_EP2.7x2.7mm, symbol Interface_USB:STUSB4500QTR
- removed U6: XC6206P272MR, Package_TO_SOT_SMD:SOT-23-3, symbol Liner-regulator_AOKI:NJM_TO-252
- removed U7: ESP32-WROOM-32, RF_Module:ESP32-WROOM-32, symbol RF_Module:ESP32-WROOM-32
- added D5, D6, D7: SS54, Diode_SMD:D_SMA, symbol Device:D_Schottky
- added H2, H3, H4: MountingHole, MountingHole:MountingHole_3.2mm_M3, symbol Mechanical:MountingHole
- added J3: Conn_02x03_Odd_Even, Connector_PinHeader_2.54mm:PinHeader_2x03_P2.54mm_Vertical_SMD, symbol Connector_Generic:Conn_02x03_Odd_Even
- added T6: PTS_1.5_2, 0_UGOKU-One_Lib:PTS_1.5_2, symbol pts_1.5_2:PTS_1.5_2
- added U5: ESP32-WROOM-32E, RF_Module:ESP32-WROOM-32D, symbol RF_Module:ESP32-WROOM-32E
- C1, C5: value 10μF -> 22μF; footprint Capacitor_SMD:C_0805_2012Metric -> Capacitor_SMD:C_0603_1608Metric
- C10, C11: footprint Capacitor_SMD:C_0805_2012Metric -> Capacitor_SMD:C_0603_1608Metric
- C6: value 10μF -> 0.1μF; footprint Capacitor_SMD:C_0805_2012Metric -> Capacitor_SMD:C_0603_1608Metric
- C7, C8: value 10μF -> 0.1uF; footprint Capacitor_SMD:C_0805_2012Metric -> Capacitor_SMD:C_0603_1608Metric
- D2, D3, D4: value D_TVS -> LESD5D5.0CT1G; footprint (none) -> Diode_SMD:D_SOD-523
- H1: footprint (none) -> MountingHole:MountingHole_3.2mm_M3
- J2: value Conn_02x03_Odd_Even -> SERVO; footprint Connector_PinHeader_2.54mm:PinHeader_2x03_P2.54mm_Vertical -> Connector_PinHeader_2.54mm:PinHeader_2x03_P2.54mm_Vertical_SMD
- SW1: footprint MultiBoardMini_Libraries:SW_TL3301FF160QG -> Button_Switch_SMD:SW_Push_1P1T_NO_Vertical_Wuerth_434133025816
- SW4, SW6: footprint (none) -> Button_Switch_SMD:SW_Push_1P1T_NO_Vertical_Wuerth_434133025816
- U1: value K7803-500R3 -> AMS1117-3.3; footprint MultiBoardMini_Libraries:M78AR -> Package_TO_SOT_SMD:SOT-223-3_TabPin2
- U4: value K7805-1000R3 -> K7805M-1000R3; footprint MultiBoardMini_Libraries:M78AR -> 0_UGOKU-One_Lib:M78AR
Connections:
- net +3V3: now also U5.2 (VDD)
- net 5V: now also D5.1 (K), D6.1 (K), D7.1 (K), J3.1 (Pin_1), J3.2 (Pin_2)
- net BAT_5V: now also D6.2 (A)
- net EN: now also U5.3 (EN)
- net GND: now also C7.1, SW4.1, T6.P$2, U5.1 (GND), U5.15 (GND), U5.38 (GND), U5.39 (GND); no longer C7.2, SW4.2
- net IO0: now also C7.2, SW4.2, U5.25 (IO0)
- net MOT_PWR: now also J3.4 (Pin_4)
- net PWR: now also J3.5 (Pin_5), J3.6 (Pin_6), T6.P$1
- net RXD: now also U5.34 (RXD0/IO3)
- net SERVO_PWR: now also J3.3 (Pin_3)
- net TXD: now also U5.35 (TXD0/IO1)
- net USB_5V: now also D2.2 (A2), P1.A4 (VBUS), P1.A9 (VBUS), P1.B4 (VBUS), P1.B9 (VBUS), R14.2, D5.2 (A)
- net LED1: now reaches L2.2 (A)
- net LED1: now also U5.24 (IO2)
- net at C11.1, U4.3 (Vout): now also D7.2 (A)
- net LED2: now reaches L3.2 (A)
- net LED2: now also U5.28 (IO17)
- net SERVO2: now reaches J2.5 (Pin_5)
- net SERVO2: now also U5.23 (IO15)
- net SERVO1: now reaches J2.6 (Pin_6)
- net SERVO1: now also U5.13 (IO14)
- net MD1_IN2: now reaches U3.2 (IN2)
- net MD1_IN2: now also U5.29 (IO5)
- net MD1_IN1: now reaches U3.3 (IN1)
- net MD1_IN1: now also U5.26 (IO4)
- net MD2_IN2: now reaches U8.2 (IN2)
- net MD2_IN2: now also U5.16 (IO13)
- net MD2_IN1: now reaches U8.3 (IN1)
- net MD2_IN1: now also U5.14 (IO12)
- no-connect marks 51 -> 18
Other:
- moved on the sheet: C7, C8, H1, J4, J5, J6, JP1, JP2, JP3, L1, L2, L3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

Commit message: Add IMU, FET
Parts:
- removed J4, J5, J6: 14110413001000, 0_UGOKU-One_Lib:14110413001000, symbol 0_14110413001000:14110413001000
- removed JP1, JP2, JP3: Jumper_NC_Dual, Jumper:SolderJumper-3_P2.0mm_Open_TrianglePad1.0x1.5mm, symbol Device:Jumper_NC_Dual
- removed SW1: PF1, Button_Switch_SMD:SW_Push_1P1T_NO_Vertical_Wuerth_434133025816, symbol Switch:SW_Push
- removed SW5: SW_Push_DPDT, MultiBoardMini_Libraries:SSSS213202, symbol Switch:SW_Push_DPDT
- added C12: 0.1uF, Capacitor_SMD:C_0603_1608Metric, symbol Device:C
- added C13, C14, C15, C4: 0.1uF, Capacitor_SMD:C_0402_1005Metric, symbol Device:C
- added J1, J7: ENC/IO, 0_UGOKU-One_Lib:14110513001000, symbol 0_14110513001000:14110513001000
- added J4: 14110213001000, 14110213001000, symbol 0_14110213001000:14110213001000
- added J8: DAC, 0_UGOKU-One_Lib:14110513001000, symbol 0_14110513001000:14110513001000
- added J9: ADC, 0_UGOKU-One_Lib:14110513001000, symbol 0_14110513001000:14110513001000
- added L4: LED, LED_SMD:LED_0805_2012Metric_Pad1.15x1.40mm_HandSolder, symbol Device:LED
- added Q1: NMOS, 0_UGOKU-One_Lib:SOT-23F, symbol Simulation_SPICE:NMOS
- added R21, R22, R23: 10k, Resistor_SMD:R_0603_1608Metric, symbol Device:R
- added R24: 100, Resistor_SMD:R_0603_1608Metric, symbol Device:R
- added R7: 1k, Resistor_SMD:R_0603_1608Metric, symbol Device:R
- added SW2: SW_SPDT, 0_UGOKU-One_Lib:SW_SS-12M11G5, symbol Switch:SW_SPDT
- added SW3, SW5: SW_Slide_DPDT, 0_UGOKU-One_Lib:SSSS213202, symbol Switch:SW_Slide_DPDT
- added U6: BMM150, Package_CSP:WLCSP-12_1.56x1.56mm_P0.4mm, symbol Sensor_Magnetic:BMM150
- added U7: BMI270, 0_UGOKU-One_Lib:XDCR_BMI270, symbol BMI270:BMI270
- C2: value C -> 22uF; footprint (none) -> Capacitor_SMD:C_0603_1608Metric
- C3: value C -> 0.1uF; footprint (none) -> Capacitor_SMD:C_0402_1005Metric
- C6: footprint Capacitor_SMD:C_0603_1608Metric -> Capacitor_SMD:C_0402_1005Metric
- R13: value 10k -> 2K
- R14: value 10k -> 22.1k
- R15: value 10k -> 47.5k
- U2: footprint 0_UGOKU-One_Lib:QFN50P500X500X80-29N -> 0_UGOKU-One_Lib:IC_CP2102N-A02-GQFN28R
- U5: footprint RF_Module:ESP32-WROOM-32D -> RF_Module:ESP32-WROOM-32E
Connections:
- net +3V3: now also R21.1, R22.1, SW5.2 (B), SW5.5 (B); no longer C10.1, U1.3 (Vout)
- net 5V: now also J1.3, J7.3, J8.3, J9.3
- net BAT_5V: now also SW2.2 (B); no longer D6.2 (A)
- net EN: now also C12.2, R21.2
- net GND: now also P1.A1 (GND), P1.A12 (GND), P1.B1 (GND), P1.B12 (GND), C12.1, C13.2, C14.2, C15.2, C4.2, J1.1, J7.1, J8.1, J9.1, Q1.3 (S), R23.2, R7.1, SW3.3 (C), SW3.4 (A), U6.A5 (CSB), U6.C1 (SDO), U6.C5 (GND), U6.E1 (GND), U6.E3 (GND), U7.1 (SDO), U7.6 (GNDIO), U7.7 (GND)
- net LED1: now also U5.26 (IO4); no longer U5.24 (IO2)
- net LED2: now also U5.37 (IO23); no longer U5.28 (IO17)
- net MD1_IN1: now also U5.29 (IO5); no longer U5.26 (IO4)
- net MD1_IN2: now also U5.16 (IO13); no longer U5.29 (IO5)
- net MD2_IN1: now also U5.8 (IO32); no longer U5.14 (IO12)
- net MD2_IN2: now also U5.9 (IO33); no longer U5.16 (IO13)
- net MOT_PWR: now also J4.1
- net SERVO2: now also U5.12 (IO27); no longer U5.23 (IO15)
- net IO25: now reaches U5.10 (IO25)
- net IO25: now also J8.4
- net IO26: now reaches U5.11 (IO26)
- net IO26: now also J8.5
- net LED3: now reaches U5.27 (IO16)
- net LED3: now also L4.2 (A)
- net IO18: now reaches U5.30 (IO18)
- net IO18: now also J1.4
- net IO19: now reaches U5.31 (IO19)
- net IO19: now also J1.5
- net SDA: now reaches U5.33 (IO21)
- net SDA: now also U7.14 (SDX)
- net SCL: now reaches U5.36 (IO22)
- net SCL: now also U7.13 (SCX)
- net SENS_VP: now reaches U5.4 (SENSOR_VP)
- net SENS_VP: now also J9.5
- net SENS_VN: now reaches U5.5 (SENSOR_VN)
- net SENS_VN: now also J9.4
- net IO34: now reaches U5.6 (IO34)
- net IO34: now also J7.4
- net IO35: now reaches U5.7 (IO35)
- net IO35: now also J7.5
- new net: D6.2 (A), SW2.3 (C)
- new net: U6.B4 (SDI), U7.2 (ASDX)
- new net: U6.A3 (SCK), U7.3 (ASCX)
- new net: L4.1 (K), R7.2
- new net: J4.2, Q1.1 (D)
- new net: Q1.2 (G), R23.1, R24.1
- new net +3V3_IMU: C13.1, C14.1, C15.1, C4.1, SW5.3 (C), SW5.4 (A), U6.A1 (PS), U6.B2 (VDDIO), U6.E5 (VDD), U7.12 (CSB), U7.5 (VDDIO), U7.8 (VDD)
- new net 3V3: C10.1, J1.2, J7.2, J8.2, J9.2, U1.3 (Vout)
- new net IO17: R24.2, U5.28 (IO17)
- new net Slide_SW: R22.2, SW3.2 (B), SW3.5 (B), U5.23 (IO15)
- no-connect marks 18 -> 23
Other:
- moved on the sheet: C7, D6, SW4

Commit message: power layout draft
Parts:
- added C16, C19: 10μF, Capacitor_SMD:C_0805_2012Metric, symbol Device:C
- added C17, C18: 0.1μF, Capacitor_SMD:C_0402_1005Metric, symbol Device:C
- added D8: SS54, Diode_SMD:D_SMA, symbol Device:D_Schottky
- C12, C7, C8: footprint Capacitor_SMD:C_0603_1608Metric -> Capacitor_SMD:C_0402_1005Metric
- J4: footprint 14110213001000 -> 0_UGOKU-One_Lib:14010213102000
- R13, R14, R15, R16, R17, R18, R19, R21, R22, R23, R24: footprint Resistor_SMD:R_0603_1608Metric -> Resistor_SMD:R_0402_1005Metric
Connections:
- net +3V3 is gone; now on net 3V3: C2.1, C3.1, C5.1, C6.1, L1.2 (A), R13.2, R21.1, R22.1, SW5.2 (B), SW5.5 (B), U2.6 (VDD), U2.7 (VREGIN), U5.2 (VDD)
- net +5V: no longer U3.4 (VREF)
- net 5V: now also U3.4 (VREF)
- net GND: now also C16.2, C17.2, C18.2, C19.2
- net MOT_PWR: now also C16.1, C17.1, C18.1, C19.1, D8.1 (K)
- net MD1_OUT1: now reaches T4.P$1, U3.6 (OUT1)
- net MD1_OUT2: now reaches T4.P$2, U3.8 (OUT2)
- net at J4.2, Q1.1 (D): now also D8.2 (A)
- net MD2_OUT1: now reaches T5.P$1, U8.6 (OUT1)
- net MD2_OUT2: now reaches T5.P$2, U8.8 (OUT2)
- net +3V3_IMU renamed 3V3_IMU
- no-connect marks 23 -> 33
Other:
- moved on the sheet: C5, C6, J4, Q1, R23, R24, U8

Commit message: Power:near complete
Connections:
- net +5V is gone; now on net 3V3: U8.4 (VREF)
- net 3V3: now also U3.4 (VREF)
- net 3V3_IMU: now also SW5.6 (A); no longer SW5.4 (A)
- net 5V: no longer U3.4 (VREF)
- net BAT_5V: now also SW2.3 (C); no longer SW2.2 (B)
- net GND: now also SW3.6; no longer SW3.4 (A)
- net LED2: now also U5.27 (IO16); no longer U5.37 (IO23)
- net LED3: now also U5.37 (IO23); no longer U5.27 (IO16)
- net SENS_VN: now also J9.5; no longer J9.4
- net SENS_VP: now also J9.4; no longer J9.5
- net at D6.2 (A): now also SW2.2 (B); no longer SW2.3 (C)
Other:
- moved on the sheet: BT1, C1, C10, C11, C12, C13, C14, C15, C16, C17, C18, C19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

Commit message: Almost done
Parts:
- removed T4, T6: PTS_1.5_2, 0_UGOKU-One_Lib:PTS_1.5_2, symbol pts_1.5_2:PTS_1.5_2
- removed T5: MultiBoardMini_Libraries:PTS_1.5_2, 0_UGOKU-One_Lib:PTS_1.5_2, symbol pts_1.5_2:PTS_1.5_2
- added J10, J12, J6: Conn_01x02, 0_UGOKU-One_Lib:PTS_1.5_2, symbol Connector_Generic:Conn_01x02
- added J5: Conn_01x05, Connector_PinHeader_2.54mm:PinHeader_1x05_P2.54mm_Vertical, symbol Connector_Generic:Conn_01x05
- added R27, R28: 10k, Resistor_SMD:R_0402_1005Metric, symbol Device:R
- L2: value LED -> IO2
- U4: value K7805M-1000R3 -> K7805M/M78AR05
Connections:
- net 3V3: now also L2.2 (A), L3.2 (A), L4.2 (A), J5.4 (Pin_4), R27.1, R28.1
- net 5V: now also J5.3 (Pin_3)
- net GND: now also J12.1 (Pin_1), J5.5 (Pin_5); no longer R5.1, R6.1, R7.1
- net IO17: now also J7.5; no longer R24.2
- net IO18: now also J1.5; no longer J1.4
- net IO19: now also J1.4; no longer J1.5
- net IO34: now also J5.2 (Pin_2); no longer J7.4
- net IO35: now also J5.1 (Pin_1); no longer J7.5
- net LED1: now also R5.1, U5.24 (IO2); no longer L2.2 (A), U5.26 (IO4)
- net LED2: now also R6.1, U5.26 (IO4); no longer L3.2 (A), U5.27 (IO16)
- net LED3: now also R7.1; no longer L4.2 (A)
- net MD1_IN1: now also U5.8 (IO32), U8.3 (IN1); no longer U3.3 (IN1), U5.29 (IO5)
- net MD1_IN2: now also U5.9 (IO33), U8.2 (IN2); no longer U3.2 (IN2), U5.16 (IO13)
- net MD2_IN1: now also U3.3 (IN1), U5.29 (IO5); no longer U5.8 (IO32), U8.3 (IN1)
- net MD2_IN2: now also U3.2 (IN2), U5.16 (IO13); no longer U5.9 (IO33), U8.2 (IN2)
- net PWR: now also J12.2 (Pin_2)
- net SCL: now also R27.2
- net SDA: now also R28.2
- net FET_SW: now reaches U5.14 (IO12)
- net FET_SW: now also R24.2
- net IO25 renamed DAC1
- net IO26 renamed DAC2
- net MD1_OUT1: no longer names the net of U3.6 (OUT1)
- net MD1_OUT1: now also J6.1 (Pin_1)
- net MD1_OUT2: no longer names the net of U3.8 (OUT2)
- net MD1_OUT2: now also J6.2 (Pin_2)
- net MD2_OUT1: no longer names the net of U8.6 (OUT1)
- net MD2_OUT1: now also J10.1 (Pin_1)
- net MD2_OUT2: no longer names the net of U8.8 (OUT2)
- net MD2_OUT2: now also J10.2 (Pin_2)
- new net IO16: J7.4, U5.27 (IO16)
Other:
- moved on the sheet: C14, C15, L1, L2, L3, L4, R4, R5, R6, R7, U7
